Commit message: con navegacion

File: urdf/tracer2.urdf (robot description, URDF)
Before this commit: robot tracer2, 10 links, 9 joints
Links:
- added link imu_link, mass 1e-5; collision box size=0.2 0.2 0.05; visual box size=0.1 0.1 0.05
Joints:
- added joint imu_joint: type fixed, parent base_link, child imu_link, origin xyz=0 0 0.15 rpy=0 0 0
- joint rslidar_joint: origin xyz=0.2125 0 0.19 rpy=0 0 0 -> xyz=0.2125 0 0.20 rpy=0 0 0

Commit message: Cambio Nombre

File: urdf/tracer2.urdf (robot description, URDF)
Before this commit: robot tracer2, 11 links, 10 joints
Links:
- link apoyo_derecho_delantero_Link: geometry collision mesh filename=package://SocialTech-Gazebo/meshes/apoyo_derecho_delantero_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; visual mesh filename=package://SocialTech-Gazebo/meshes/apoyo_derecho_delantero_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
- link apoyo_derecho_trasero_Link: geometry collision mesh filename=package://SocialTech-Gazebo/meshes/apoyo_derecho_trasero_Li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; visual mesh filename=package://SocialTech-Gazebo/meshes/apoyo_derecho_trasero_Li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
- link apoyo_izquierdo_delantero_Link: geometry collision mesh filename=package://SocialTech-Gazebo/meshes/apoyo_izquierdo_delanter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; visual mesh filename=package://SocialTech-Gazebo/meshes/apoyo_izquierdo_delanter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
- link apoyo_izquierdo_trasero_Link: geometry collision mesh filename=package://SocialTech-Gazebo/meshes/apoyo_izquierdo_trasero_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; visual mesh filename=package://SocialTech-Gazebo/meshes/apoyo_izquierdo_trasero_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
- link base_link: geometry collision mesh filename=package://SocialTech-Gazebo/meshes/base_link.STL; visual mesh filename=package://SocialTech-Gazebo/meshes/base_link.STL
- link rueda_derecha_Link: geometry collision mesh filename=package://SocialTech-Gazebo/meshes/rueda_derecha_Link.STL; visual mesh filename=package://SocialTech-Gazebo/meshes/rueda_derecha_Link.STL
- link rueda_izquierda_Link: geometry collision mesh filename=package://SocialTech-Gazebo/meshes/rueda_izquierda_Link.STL; visual mesh filename=package://SocialTech-Gazebo/meshes/rueda_izquierda_Link.STL
